Commit message: 更新urdf、geni_craner_hardware硬件驱动代码；新增easy_handeye2 easy_handeye2_msgs；新增scripts脚本目录

File: geni_craner_description/urdf/geni_craner.ros2_control.xacro (robot description, xacro)
@@ -19,6 +19,6 @@
         <param name="can_interface">can1</param>
         <param name="direction">-1.0</param>
-        <param name="lower_limit">-1.57</param>
-        <param name="upper_limit">1.57</param>
+        <param name="lower_limit">-3.1415</param>
+        <param name="upper_limit">3.1415</param>
         <command_interface name="position"/>
         <state_interface name="position"/>
@@ -31,6 +31,7 @@
         <param name="can_interface">can1</param>
         <param name="direction">-1.0</param>
-        <param name="lower_limit">-1.57</param>
-        <param name="upper_limit">1.57</param>
+        <param name="lower_limit">-2.0944</param>
+        <param name="upper_limit">2.0944</param>
+        <param name="kp">200</param>
         <command_interface name="position"/>
         <state_interface name="position"/>
@@ -43,6 +44,6 @@
         <param name="can_interface">can0</param>
         <param name="direction">-1.0</param>
-        <param name="lower_limit">-1.57</param>
-        <param name="upper_limit">1.57</param>
+        <param name="lower_limit">-3.1415</param>
+        <param name="upper_limit">3.1415</param>
         <command_interface name="position"/>
         <state_interface name="position"/>
@@ -55,6 +56,6 @@
         <param name="can_interface">can0</param>
         <param name="direction">-1.0</param>
-        <param name="lower_limit">-1.57</param>
-        <param name="upper_limit">1.57</param>
+        <param name="lower_limit">-1.658</param>
+        <param name="upper_limit">1.658</param>
         <command_interface name="position"/>
         <state_interface name="position"/>
@@ -67,6 +68,6 @@
         <param name="can_interface">can0</param>
         <param name="direction">-1.0</param>
-        <param name="lower_limit">-1.57</param>
-        <param name="upper_limit">1.57</param>
+        <param name="lower_limit">-3.1415</param>
+        <param name="upper_limit">3.1415</param>
         <command_interface name="position"/>
         <state_interface name="position"/>
@@ -79,6 +80,6 @@
         <param name="can_interface">can0</param>
         <param name="direction">-1.0</param>
-        <param name="lower_limit">-1.57</param>
-        <param name="upper_limit">1.57</param>
+        <param name="lower_limit">-1.658</param>
+        <param name="upper_limit">1.658</param>
         <command_interface name="position"/>
         <state_interface name="position"/>
@@ -91,6 +92,6 @@
         <param name="can_interface">can0</param>
         <param name="direction">-1.0</param>
-        <param name="lower_limit">-1.57</param>
-        <param name="upper_limit">1.57</param>
+        <param name="lower_limit">-3.1415</param>
+        <param name="upper_limit">3.1415</param>
         <command_interface name="position"/>
         <state_interface name="position"/>

File: geni_craner_description/urdf/geni_craner.urdf (robot description, URDF)
Before this commit: robot geni_craner, 10 links, 9 joints
Joints:
- joint joint1: limit lower=-1.57 upper=1.57 effort=6 velocity=5 -> lower=-3.1415 upper=3.1415 effort=6 velocity=5
- joint joint2: limit lower=-1.57 upper=1.57 effort=20 velocity=5 -> lower=-2.0944 upper=2.0944 effort=20 velocity=5
- joint joint3: limit lower=-1.57 upper=1.57 effort=5 velocity=5 -> lower=-3.1415 upper=3.1415 effort=5 velocity=5
- joint joint4: limit lower=-1.57 upper=1.57 effort=5 velocity=5 -> lower=-1.658 upper=1.658 effort=5 velocity=5
- joint joint5: limit lower=-1.57 upper=1.57 effort=5 velocity=5 -> lower=-3.1415 upper=3.1415 effort=5 velocity=5
- joint joint6: limit lower=-1.57 upper=1.57 effort=5 velocity=5 -> lower=-1.658 upper=1.658 effort=5 velocity=5
- joint joint7: limit lower=-3.14 upper=3.14 effort=5 velocity=5 -> lower=-3.1415 upper=3.1415 effort=5 velocity=5
